Commit message: reorganised repository for a new package
Signed-off-by: lkw303 <lkw303@gmail.com>

File: hub/urdf/hub.urdf.xacro (robot description, xacro)
@@ -12,5 +12,5 @@
         <inertial>
             <inertia ixx="0.0" ixy="0.0" ixz="0.0" iyy="0.0" iyz="0.0" izz="0.0"/>
-            <mass value="0.1"/>
+            <mass value="1"/>
         </inertial>
     </link>
@@ -36,5 +36,5 @@
 					  <inertial>
             	<inertia ixx="0.000" ixy="0.0" ixz="0.0" iyy="0.0" iyz="0.0" izz="0.00"/>
-            	<mass value="0.01"/>
+            	<mass value="1"/>
         		</inertial>
         </link>
@@ -59,6 +59,6 @@
         </visual>
         <inertial>
-            <inertia ixx="0.001" ixy="0.0" ixz="0.0" iyy="0.0" iyz="0.0" izz="0.001"/>
-            <mass value="2"/>
+            <inertia ixx="0.0" ixy="0.0" ixz="0.0" iyy="0.0" iyz="0.0" izz="0.0"/>
+            <mass value="0.01"/>
             <!-- <mass value="${al_density*ext_width*ext_height*x_axis_arm_length}"/> -->
         </inertial>
@@ -69,5 +69,5 @@
         <child link="x_axis_arm"/>
         <axis xyz="1 0 0"/>
-         <limit effort="10000" lower="-${hub_height/2}" upper="${hub_height/2}" velocity="1" />
+         <limit effort="10" lower="-${hub_height/2}" upper="${hub_height/2}" velocity="0.1" />
     </joint>
   	<ros2_control name="GazeboSystem" type="system">
@@ -96,6 +96,6 @@
         </visual>
         <inertial>
-            <inertia ixx="0.001" ixy="0.0" ixz="0.0" iyy="0.0" iyz="0.0" izz="0.001"/>
-            <mass value="0.5"/>
+            <inertia ixx="0.0" ixy="0.0" ixz="0.0" iyy="0.0" iyz="0.0" izz="0.0"/>
+            <mass value="0.01"/>
         </inertial>
     </link>
@@ -105,5 +105,5 @@
         <origin xyz="-${ext_width} 0.0 0.0"/>
         <axis xyz="0 0 1"/>
-        <limit effort="10000" lower="-${hub_width/2}" upper="${hub_width/2}" velocity="0.01" />
+        <limit effort="10" lower="-${hub_width/2}" upper="${hub_width/2}" velocity="0.1" />
     </joint>
   	<ros2_control name="GazeboSystem" type="system">
